Commit message: Fixing base rotation

File: urdf/phantomx_turret.urdf.xacro (robot description, xacro)
@@ -16,5 +16,5 @@
   <link name="base_link"/>
   <base_mount parent="base_link" name="base_mount" color="Gray" >
-      <origin xyz="0 0 0"/>
+      <origin xyz="0 0 0" rpy="${M_PI/2} 0 0"/>
   </base_mount>
   <!-- AX-12A Pan !-->

Commit message: Fixed AX-12A rotation

File: urdf/phantomx_turret.urdf.xacro (robot description, xacro)
@@ -20,5 +20,5 @@
   <!-- AX-12A Pan !-->
   <AX12A_fixed parent="base_mount_link" name="pan_servo">
-    <origin xyz="-2e-6 0.0763 -9e-6" rpy="${M_PI/2} 0 0"/>
+    <origin xyz="-2e-6 0.0763 -9e-6" rpy="${-M_PI/2} 0 0"/>
   </AX12A_fixed>
 </robot>

Commit message: Added limits

File: urdf/phantomx_turret.urdf.xacro (robot description, xacro)
@@ -2,4 +2,11 @@
 <robot name="phantomx_turret" xmlns:xacro="http://ros.org/wiki/xacro">
   <xacro:include filename="$(find phantomx_turret)/urdf/pan_tilt_hardware.xacro"/>
+  <!-- angle limits in rad ~ +/- 150 deg !-->
+  <xacro:property name="ax12_llimit" value="${-(5.0/6.0)*M_PI}"/>
+  <xacro:property name="ax12_ulimit" value="${(5.0/6.0)*M_PI}"/>
+  <!-- vlimit in rad/s ~(0.111rpm * 1023) !-->
+  <xacro:property name="ax12_vlimit" value="11.891242339515"/>
+  <!-- elimit in N m !-->
+  <xacro:property name="ax12_elimit" value="1.5"/>
   <material name="White">
     <color rgba="0.87 0.90 0.87 1.0"/>
@@ -22,5 +29,7 @@
     <origin xyz="-2e-6 0.0763 -9e-6" rpy="${-M_PI/2} 0 0"/>
   </AX12A_fixed>
-  <interbotix_F3_bracket_revolute parent="pan_servo_link" name="pan_F3">
+  <interbotix_F3_bracket_revolute parent="pan_servo_link" name="pan_F3" color="Gray"
+                                  elimit="${ax12_elimit}" vlimit="${ax12_vlimit}"
+                                  llimit="${ax12_llimit}" ulimit="${ax12_ulimit}">
     <origin xyz="-2e-6 0.09724 -9e-6" rpy="0 0 0"/>
   </interbotix_F3_bracket_revolute>

Commit message: Added pan servo

File: urdf/phantomx_turret.urdf.xacro (robot description, xacro)
@@ -34,3 +34,7 @@
     <origin xyz="0 0 0.02094" rpy="0 0 ${M_PI/2}"/>
   </interbotix_F3_bracket_revolute>
+  <!-- AX-12A Pan !-->
+  <AX12A_fixed parent="interbotix_F3_bracket_revolute_link" name="tilt_servo">
+    <origin xyz="0 0 0.0415" rpy="0 0 0"/>
+  </AX12A_fixed>
 </robot>

Commit message: Added gitignore file Finished adding tilt servo

File: urdf/phantomx_turret.urdf.xacro (robot description, xacro)
@@ -35,6 +35,6 @@
   </interbotix_F3_bracket_revolute>
   <!-- AX-12A Pan !-->
-  <AX12A_fixed parent="interbotix_F3_bracket_revolute_link" name="tilt_servo">
-    <origin xyz="0 0 0.0415" rpy="0 0 0"/>
+  <AX12A_fixed parent="pan_F3_link" name="tilt_servo">
+    <origin xyz="0 0 0.0415" rpy="${M_PI/2} 0 0"/>
   </AX12A_fixed>
 </robot>

Commit message: Fixed pan servo position

File: urdf/phantomx_turret.urdf.xacro (robot description, xacro)
@@ -29,5 +29,5 @@
                         elimit="${ax12_elimit}" vlimit="${ax12_vlimit}"
                         llimit="${ax12_llimit}" ulimit="${ax12_ulimit}">
-    <origin xyz="-2e-6 0.0763 -9e-6" rpy="${-M_PI/2} 0 0"/>
+    <origin xyz="-2e-6 -9e-6 0.0763" rpy="0 0 0"/>
   </AX12A_compound_fixed>
 </robot>

Commit message: Added tilt servo

File: urdf/phantomx_turret.urdf.xacro (robot description, xacro)
@@ -34,8 +34,8 @@
     <origin xyz="0 0 0.02094" rpy="0 0 0"/>
   </interbotix_F3_bracket_fixed>
-  <AX12A_compound_fixed parent="base_mount_link" name="pan_servo"
+  <AX12A_compound_fixed parent="pan_F3_link" name="tilt_servo"
                         elimit="${ax12_elimit}" vlimit="${ax12_vlimit}"
                         llimit="${ax12_llimit}" ulimit="${ax12_ulimit}">
-    <origin xyz="0 0 0.0415" rpy="${M_PI/2} 0 0"/>
+    <origin xyz="0 0 0.0415" rpy="${M_PI/2} 0 ${M_PI/2}"/>
   </AX12A_compound_fixed>
 </robot>

Commit message: Corrected F2 bracket position

File: urdf/phantomx_turret.urdf.xacro (robot description, xacro)
@@ -40,5 +40,5 @@
   </AX12A_compound_fixed>
   <interbotix_F2_bracket_fixed parent="tilt_servo_link" name="pan_F2" color="Gray">
-    <origin xyz="-3.601e-7 0.017175 -0.002002" rpy="0 0 0"/>
+    <origin xyz="-0.002002 0.017175 -3.601e-7" rpy="0 0 0"/>
   </interbotix_F2_bracket_fixed>
 </robot>

Commit message: More work

File: urdf/phantomx_turret.urdf.xacro (robot description, xacro)
@@ -21,6 +21,7 @@
     <color rgba="0.22 0.32 0.14 1.0"/>
   </material>
-  <link name="base_link"/>
-  <base_mount parent="base_link" name="base_mount" color="Gray" >
+  <!-- Used for fixing robot to Gazebo 'base_link' -->
+  <link name="world"/>
+  <base_mount parent="world" name="base_mount" color="Gray" >
       <origin xyz="0 0 0" rpy="0 0 0"/>
   </base_mount>

Commit message: Fixed rviz stuff

File: urdf/phantomx_turret.urdf.xacro (robot description, xacro)
@@ -21,7 +21,13 @@
     <color rgba="0.22 0.32 0.14 1.0"/>
   </material>
-  <!-- Used for fixing robot to Gazebo 'base_link' -->
-  <link name="world"/>
-  <base_mount parent="world" name="base_mount" color="Gray" >
+  <!-- ros_control plugin -->
+  <gazebo>
+    <plugin name="gazebo_ros_control" filename="libgazebo_ros_control.so">
+      <robotNamespace>/phantomx_turret</robotNamespace>
+      <robotSimType>gazebo_ros_control/DefaultRobotHWSim</robotSimType>
+    </plugin>
+  </gazebo>
+  <link name="base_link"/>
+  <base_mount parent="base_link" name="base_mount" color="Gray" >
       <origin xyz="0 0 0" rpy="0 0 0"/>
   </base_mount>
