Commit message: Added base

File: urdf/pan_tilt_hardware.xacro (robot description, xacro)
@@ -1 +1,39 @@
 <?xml version="1.0"?>
+<robot xmlns:xacro="http://ros.org/wiki/xacro">
+  <xacro:property name="M_PI" value="3.14159"/>
+  <xacro:property name="M_SCALE" value="0.001"/>
+  <xacro:macro name="base_mount" params="parent name color *origin">
+    <joint name="${name}_joint" type="fixed">
+      <insert_block name="origin"/>
+        <parent link="${parent}"/>
+        <child link="${name}_link"/>
+    </joint>
+    <link name="${name}_link">
+      <inertial>
+        <mass value="0.21328"/>
+        <origin xyz="0.00199427 0.0257168 0.00107065"/>
+        <inertia ixx="0.0003798" ixy="-6.70148E-7" ixz="-5.778745E-6"
+                 iyy="0.0006116" iyz="-8.17711E-7"
+                 izz="0.000379"/>
+      </inertial>
+      <visual>
+        <origin xyz="0 0 0" rpy="0 0 0"/>
+        <geometry>
+          <mesh filename="package://phantomx_turret/meshes/base.stl" scale="${M_SCALE} ${M_SCALE} ${M_SCALE}"/>
+        </geometry>
+        <material name="${color}"/>
+      </visual>
+      <collision>
+        <origin xyz="0 0 0" rpy="0 0 0"/>
+        <geometry>
+          <box size="0 0 0"/>
+        </geometry>
+      </collision>
+    </link>
+    <gazebo reference="${name}_link">
+      <material>Gazebo/${color}</material>
+      <selfCollide>true</selfCollide>
+      <gravity>true</gravity>
+    </gazebo>
+  </xacro:macro>
+</robot>

Commit message: Fixed capitalization

File: urdf/pan_tilt_hardware.xacro (robot description, xacro)
@@ -20,5 +20,5 @@
         <origin xyz="0 0 0" rpy="0 0 0"/>
         <geometry>
-          <mesh filename="package://phantomx_turret/meshes/base.stl" scale="${M_SCALE} ${M_SCALE} ${M_SCALE}"/>
+          <mesh filename="package://phantomx_turret/meshes/Base.stl" scale="${M_SCALE} ${M_SCALE} ${M_SCALE}"/>
         </geometry>
         <material name="${color}"/>

Commit message: Modified rotation

File: urdf/pan_tilt_hardware.xacro (robot description, xacro)
@@ -18,5 +18,5 @@
       </inertial>
       <visual>
-        <origin xyz="0 0 0" rpy="0 0 0"/>
+        <origin xyz="0 0 0" rpy="${M_PI/2} 0 0"/>
         <geometry>
           <mesh filename="package://phantomx_turret/meshes/Base.stl" scale="${M_SCALE} ${M_SCALE} ${M_SCALE}"/>

Commit message: Adding AX-12A

File: urdf/pan_tilt_hardware.xacro (robot description, xacro)
@@ -37,3 +37,59 @@
     </gazebo>
   </xacro:macro>
+  <xacro:macro name="AX12A_fixed" params="parent name *origin">
+    <joint name="${name}_joint" type="fixed">
+      <xacro:insert_block name="origin"/>
+      <parent link="${parent}"/>
+      <child link="${name}_link"/>
+    </joint>
+    <link name="${name}_link">
+      <inertial>
+        <mass value="0.0546"/>
+        <origin xyz="-3.09266e-5 0.0774271 0.0125938"/>
+        <inertia ixx="0.0003798" ixy="-6.70148E-7" ixz="-5.778745E-6"
+                 iyy="0.0006116" iyz="-8.17711E-7"
+                 izz="0.000379"/>
+      </inertial>
+ASM0002_ASM
+Area  1.389E+04 mm^2
+Density 0.001 g / mm^3
+Mass  47.854 g
+Volume  4.279E+04 mm^3
+Physical Material (Various)
+Bounding Box
+Length   32.00 mm
+Width    40.047 mm
+Height   50.00 mm
+World X,Y,Z 0 mm, 110 mm, -1.74305e-13 mm
+Center of Mass  -0.0309266 mm, 77.4271 mm, 12.5938 mm
+Moment of Inertia at Center of Mass   (g mm^2)
+  Ixx = 1.439E+04
+  Ixy = 1.541
+  Ixz = 11.563
+  Iyx = 1.541
+  Iyy = 1.219E+04
+  Iyz = 216.221
+  Izx = 11.563
+  Izy = 216.221
+  Izz = 7768.456
+      <visual>
+        <origin xyz="0 0 0" rpy="0 0 0"/>
+        <geometry>
+          <mesh filename="package://phantomx_turret/meshes/AX-12A.stl" scale="${M_SCALE} ${M_SCALE} ${M_SCALE}"/>
+        </geometry>
+        <material name="Black"/>
+      </visual>
+      <collision>
+        <origin xyz="0 0 0" rpy="0 0 0"/>
+        <geometry>
+          <box size="0 0 0"/>
+        </geometry>
+      </collision>
+    </link>
+    <gazebo reference="${name}_link">
+      <material>Gazebo/Black</material>
+      <selfCollide>true</selfCollide>
+      <gravity>true</gravity>
+    </gazebo>
+  </xacro:macro>
 </robot>

Commit message: Adding AX-12A and pan

File: urdf/pan_tilt_hardware.xacro (robot description, xacro)
@@ -51,10 +51,4 @@
                  izz="0.000379"/>
       </inertial>
-ASM0002_ASM
-Area  1.389E+04 mm^2
-Density 0.001 g / mm^3
-Mass  47.854 g
-Volume  4.279E+04 mm^3
-Physical Material (Various)
 Bounding Box
 Length   32.00 mm
@@ -74,5 +68,5 @@
   Izz = 7768.456
       <visual>
-        <origin xyz="0 0 0" rpy="0 0 0"/>
+        <origin xyz="0 0 0" rpy="${M_PI/2} 0 0"/>
         <geometry>
           <mesh filename="package://phantomx_turret/meshes/AX-12A.stl" scale="${M_SCALE} ${M_SCALE} ${M_SCALE}"/>
@@ -83,5 +77,5 @@
         <origin xyz="0 0 0" rpy="0 0 0"/>
         <geometry>
-          <box size="0 0 0"/>
+          <box size="0.032 0.040047 0.05"/>
         </geometry>
       </collision>

File: urdf/phantomx_turret.urdf.xacro (robot description, xacro)
@@ -18,3 +18,7 @@
       <origin xyz="0 0 0"/>
   </base_mount>
+  <!-- AX-12A Pan !-->
+  <AX12A_fixed parent="base_mount_link" name="pan_servo">
+    <origin xyz="0 0.11 -1.74305e-16" rpy="0 0 0"/>
+  </AX12A_fixed>
 </robot>

Commit message: Fixing up AX-12A

File: urdf/pan_tilt_hardware.xacro (robot description, xacro)
@@ -18,5 +18,5 @@
       </inertial>
       <visual>
-        <origin xyz="0 0 0" rpy="${M_PI/2} 0 0"/>
+        <origin xyz="0 0 0" rpy="0 0 0"/>
         <geometry>
           <mesh filename="package://phantomx_turret/meshes/Base.stl" scale="${M_SCALE} ${M_SCALE} ${M_SCALE}"/>
@@ -46,27 +46,11 @@
       <inertial>
         <mass value="0.0546"/>
-        <origin xyz="-3.09266e-5 0.0774271 0.0125938"/>
-        <inertia ixx="0.0003798" ixy="-6.70148E-7" ixz="-5.778745E-6"
-                 iyy="0.0006116" iyz="-8.17711E-7"
-                 izz="0.000379"/>
+        <origin xyz="-2.89001e-5 -0.0126033 0.00112682"/>
+        <inertia ixx="1.43900e-5" ixy="1.54100e-9" ixz="1.1563e-8"
+                 iyy="1.21900e-5" iyz="2.16221e-7"
+                 izz="7.768456e-6"/>
       </inertial>
-Bounding Box
-Length   32.00 mm
-Width    40.047 mm
-Height   50.00 mm
-World X,Y,Z 0 mm, 110 mm, -1.74305e-13 mm
-Center of Mass  -0.0309266 mm, 77.4271 mm, 12.5938 mm
-Moment of Inertia at Center of Mass   (g mm^2)
-  Ixx = 1.439E+04
-  Ixy = 1.541
-  Ixz = 11.563
-  Iyx = 1.541
-  Iyy = 1.219E+04
-  Iyz = 216.221
-  Izx = 11.563
-  Izy = 216.221
-  Izz = 7768.456
       <visual>
-        <origin xyz="0 0 0" rpy="${M_PI/2} 0 0"/>
+        <origin xyz="0 0 0" rpy="0 0 0"/>
         <geometry>
           <mesh filename="package://phantomx_turret/meshes/AX-12A.stl" scale="${M_SCALE} ${M_SCALE} ${M_SCALE}"/>
@@ -75,7 +59,7 @@
       </visual>
       <collision>
-        <origin xyz="0 0 0" rpy="0 0 0"/>
+        <origin xyz="0 -0.0135 0.0010025" rpy="0 0 0"/>
         <geometry>
-          <box size="0.032 0.040047 0.05"/>
+          <box size="0.032 0.05 0.040047"/>
         </geometry>
       </collision>

File: urdf/phantomx_turret.urdf.xacro (robot description, xacro)
@@ -20,5 +20,5 @@
   <!-- AX-12A Pan !-->
   <AX12A_fixed parent="base_mount_link" name="pan_servo">
-    <origin xyz="0 0.11 -1.74305e-16" rpy="0 0 0"/>
+    <origin xyz="-2e-6 0.0763 -9e-6" rpy="${M_PI/2} 0 0"/>
   </AX12A_fixed>
 </robot>

Commit message: Fixed Rotation Added Collision for base

File: urdf/pan_tilt_hardware.xacro (robot description, xacro)
@@ -25,7 +25,19 @@
       </visual>
       <collision>
-        <origin xyz="0 0 0" rpy="0 0 0"/>
+        <origin xyz="-2e-6 0.05785 -9e-6" rpy="0 0 0"/>
         <geometry>
-          <box size="0 0 0"/>
+          <box size="0.1045 0.0049 0.1045"/>
+        </geometry>
+      </collision>
+      <collision>
+        <origin xyz="-2e-6 0.0329 -9.5e-6" rpy="0 0 0"/>
+        <geometry>
+          <box size="0.086 0.045 0.086929"/>
+        </geometry>
+      </collision>
+      <collision>
+        <origin xyz="-2e-6 0.005139 -9e-6" rpy="0 0 0"/>
+        <geometry>
+          <box size="0.178 0.010522 0.178"/>
         </geometry>
       </collision>

File: urdf/phantomx_turret.urdf.xacro (robot description, xacro)
@@ -20,5 +20,5 @@
   <!-- AX-12A Pan !-->
   <AX12A_fixed parent="base_mount_link" name="pan_servo">
-    <origin xyz="-2e-6 0.0763 -9e-6" rpy="${M_PI/2} 0 0"/>
+    <origin xyz="-2e-6 0.0763 -9e-6" rpy="$-{M_PI/2} 0 0"/>
   </AX12A_fixed>
 </robot>

Commit message: Work on adding F3 bracket

File: urdf/pan_tilt_hardware.xacro (robot description, xacro)
@@ -83,3 +83,40 @@
     </gazebo>
   </xacro:macro>
+  <xacro:macro name="interbotix_F3_bracket_revolute" params="parent name color llimit ulimit vlimit elimit *origin">
+    <joint name="${name}_joint" type="revolute">
+      <xacro:insert_block name="origin"/>
+      <axis xyz="0 1 0"/>
+      <limit effort="${elimit}" velocity="${vlimit}" lower="${llimit}" upper="${ulimit}"/>
+      <dynamics friction="0.13"/>
+      <parent link="${parent}"/>
+      <child link="${name}_link"/>
+    </joint>
+    <link name="${name}_link">
+      <inertial>
+        <mass value="0.004398"/>
+        <origin xyz="2.45363e-17 -2.45363e-17 0.00183916"/>
+        <inertia ixx="7.00046e-7" ixy="0" ixz="0"
+                 iyy="2.66739e-7" iyz="0"
+                 izz="9.31478e-7"/>
+      </inertial>
+      <visual>
+        <origin xyz="0 0 0" rpy="0 0 0"/>
+        <geometry>
+          <mesh filename="package://phantomx_turret/meshes/F3-Bracket.stl" scale="${M_SCALE} ${M_SCALE} ${M_SCALE}"/>
+        </geometry>
+        <material name="${color}"/>
+      </visual>
+      <collision>
+        <origin xyz="0 0 0" rpy="0 0 0"/>
+        <geometry>
+          <box size="0 0 0"/>
+        </geometry>
+      </collision>
+    </link>
+    <gazebo reference="${name}_link">
+      <material>Gazebo/${color}</material>
+      <selfCollide>true</selfCollide>
+      <gravity>true</gravity>
+    </gazebo>
+  </xacro:macro>
 </robot>

File: urdf/phantomx_turret.urdf.xacro (robot description, xacro)
@@ -22,3 +22,6 @@
     <origin xyz="-2e-6 0.0763 -9e-6" rpy="${-M_PI/2} 0 0"/>
   </AX12A_fixed>
+  <interbotix_F3_bracket_revolute parent="pan_servo_link" name="pan_F3">
+    <origin xyz="-2e-6 0.09724 -9e-6" rpy="0 0 0"/>
+  </interbotix_F3_bracket_revolute>
 </robot>

Commit message: Corrected F3 bracket and joint

File: urdf/pan_tilt_hardware.xacro (robot description, xacro)
@@ -86,5 +86,5 @@
     <joint name="${name}_joint" type="revolute">
       <xacro:insert_block name="origin"/>
-      <axis xyz="0 1 0"/>
+      <axis xyz="0 0 1"/>
       <limit effort="${elimit}" velocity="${vlimit}" lower="${llimit}" upper="${ulimit}"/>
       <dynamics friction="0.13"/>

File: urdf/phantomx_turret.urdf.xacro (robot description, xacro)
@@ -32,5 +32,5 @@
                                   elimit="${ax12_elimit}" vlimit="${ax12_vlimit}"
                                   llimit="${ax12_llimit}" ulimit="${ax12_ulimit}">
-    <origin xyz="-2e-6 0.09724 -9e-6" rpy="0 0 0"/>
+    <origin xyz="0 0 0.02094" rpy="0 0 ${M_PI/2}"/>
   </interbotix_F3_bracket_revolute>
 </robot>

Commit message: Trying differet approach with AX-12

File: urdf/pan_tilt_hardware.xacro (robot description, xacro)
@@ -18,5 +18,5 @@
       </inertial>
       <visual>
-        <origin xyz="0 0 0" rpy="0 0 0"/>
+        <origin xyz="0 0 0" rpy="${M_PI/2} 0 0"/>
         <geometry>
           <mesh filename="package://phantomx_turret/meshes/Base.stl" scale="${M_SCALE} ${M_SCALE} ${M_SCALE}"/>
@@ -83,4 +83,71 @@
     </gazebo>
   </xacro:macro>
+  <xacro:macro name="AX12A_compound_fixed" params="parent name *origin">
+    <joint name="${name}_body_joint" type="fixed">
+      <xacro:insert_block name="origin"/>
+      <parent link="${parent}"/>
+      <child link="${name}_link"/>
+    </joint>
+    <link name="${name}_body_link">
+      <inertial>
+        <mass value="0.052587"/>
+        <origin xyz="-3.01694e-5 -0.0131566 0.000442296"/>
+        <inertia ixx="1.3400e-05" ixy="-1.0798e-08" ixz="2.4880e-09"
+                 iyy="7.1120e-06" iyz="1.9648e-07"
+                 izz="1.1780e-05"/>
+      </inertial>
+      <visual>
+        <origin xyz="0 0 0" rpy="0 0 0"/>
+        <geometry>
+          <mesh filename="package://phantomx_turret/meshes/AX-12A-Fixed.stl" scale="${M_SCALE} ${M_SCALE} ${M_SCALE}"/>
+        </geometry>
+        <material name="Black"/>
+      </visual>
+      <collision>
+        <origin xyz="0 0 0" rpy="0 0 0"/>
+        <geometry>
+          <box size="0 0 0"/>
+        </geometry>
+      </collision>
+    </link>
+    <gazebo reference="${name}_body_link">
+      <material>Gazebo/Black</material>
+      <selfCollide>true</selfCollide>
+      <gravity>true</gravity>
+    </gazebo>
+    <joint name="${name}_horn_joint" type="revolute">
+      <origin xyz="0 0 0" rpy="0 0 0"/>
+      <axis xyz="0 0 1"/>
+      <parent link="${name}_body_link"/>
+      <child link="${name}_link"/>
+    </joint>
+    <link name="${name}_link">
+      <inertial>
+        <mass value="0.002013"/>
+        <origin xyz="2.05733e-9 -3.64002e-6 0.0167129"/>
+        <inertia ixx="1.4571e-07" ixy="5.0780e-15" ixz="-1.7060e-14"
+                 iyy="1.4591e-07" iyz="1.7000e-11"
+                 izz="7.6730e-08"/>
+      </inertial>
+      <visual>
+        <origin xyz="0 0 0" rpy="0 0 0"/>
+        <geometry>
+          <mesh filename="package://phantomx_turret/meshes/AX-12A-Rotating.stl" scale="${M_SCALE} ${M_SCALE} ${M_SCALE}"/>
+        </geometry>
+        <material name="Black"/>
+      </visual>
+      <collision>
+        <origin xyz="0 0 0" rpy="0 0 0"/>
+        <geometry>
+          <box size="0 0 0"/>
+        </geometry>
+      </collision>
+    </link>
+    <gazebo reference="${name}_link">
+      <material>Gazebo/Black</material>
+      <selfCollide>true</selfCollide>
+      <gravity>true</gravity>
+    </gazebo>
+  </xacro:macro>
   <xacro:macro name="interbotix_F3_bracket_revolute" params="parent name color llimit ulimit vlimit elimit *origin">
     <joint name="${name}_joint" type="revolute">

File: urdf/phantomx_turret.urdf.xacro (robot description, xacro)
@@ -23,18 +23,9 @@
   <link name="base_link"/>
   <base_mount parent="base_link" name="base_mount" color="Gray" >
-      <origin xyz="0 0 0" rpy="${M_PI/2} 0 0"/>
+      <origin xyz="0 0 0" rpy="0 0 0"/>
   </base_mount>
   <!-- AX-12A Pan !-->
-  <AX12A_fixed parent="base_mount_link" name="pan_servo">
+  <AX12A_compound_fixed parent="base_mount_link" name="pan_servo">
     <origin xyz="-2e-6 0.0763 -9e-6" rpy="${-M_PI/2} 0 0"/>
-  </AX12A_fixed>
-  <interbotix_F3_bracket_revolute parent="pan_servo_link" name="pan_F3" color="Gray"
-                                  elimit="${ax12_elimit}" vlimit="${ax12_vlimit}"
-                                  llimit="${ax12_llimit}" ulimit="${ax12_ulimit}">
-    <origin xyz="0 0 0.02094" rpy="0 0 ${M_PI/2}"/>
-  </interbotix_F3_bracket_revolute>
-  <!-- AX-12A Pan !-->
-  <AX12A_fixed parent="pan_F3_link" name="tilt_servo">
-    <origin xyz="0 0 0.0415" rpy="${M_PI/2} 0 0"/>
-  </AX12A_fixed>
+  </AX12A_compound_fixed>
 </robot>

Commit message: Added limits

File: urdf/pan_tilt_hardware.xacro (robot description, xacro)
@@ -83,5 +83,5 @@
     </gazebo>
   </xacro:macro>
-  <xacro:macro name="AX12A_compound_fixed" params="parent name *origin">
+  <xacro:macro name="AX12A_compound_fixed" params="parent name llimit ulimit vlimit elimit *origin">
     <joint name="${name}_body_joint" type="fixed">
       <xacro:insert_block name="origin"/>
@@ -119,4 +119,6 @@
       <origin xyz="0 0 0" rpy="0 0 0"/>
       <axis xyz="0 0 1"/>
+      <limit effort="${elimit}" velocity="${vlimit}" lower="${llimit}" upper="${ulimit}"/>
+      <dynamics friction="0.13"/>
       <parent link="${name}_body_link"/>
       <child link="${name}_link"/>

File: urdf/phantomx_turret.urdf.xacro (robot description, xacro)
@@ -26,5 +26,7 @@
   </base_mount>
   <!-- AX-12A Pan !-->
-  <AX12A_compound_fixed parent="base_mount_link" name="pan_servo">
+  <AX12A_compound_fixed parent="base_mount_link" name="pan_servo"
+                        elimit="${ax12_elimit}" vlimit="${ax12_vlimit}"
+                        llimit="${ax12_llimit}" ulimit="${ax12_ulimit}">
     <origin xyz="-2e-6 0.0763 -9e-6" rpy="${-M_PI/2} 0 0"/>
   </AX12A_compound_fixed>

Commit message: Fixed joint

File: urdf/pan_tilt_hardware.xacro (robot description, xacro)
@@ -87,5 +87,5 @@
       <xacro:insert_block name="origin"/>
       <parent link="${parent}"/>
-      <child link="${name}_link"/>
+      <child link="${name}_body_link"/>
     </joint>
     <link name="${name}_body_link">

Commit message: readding F3 bracket

File: urdf/pan_tilt_hardware.xacro (robot description, xacro)
@@ -189,3 +189,37 @@
     </gazebo>
   </xacro:macro>
+  <xacro:macro name="interbotix_F3_bracket_fixed" params="parent name color *origin">
+    <joint name="${name}_joint" type="fixed">
+      <xacro:insert_block name="origin"/>
+      <parent link="${parent}"/>
+      <child link="${name}_link"/>
+    </joint>
+    <link name="${name}_link">
+      <inertial>
+        <mass value="0.004398"/>
+        <origin xyz="2.45363e-17 -2.45363e-17 0.00183916"/>
+        <inertia ixx="7.00046e-7" ixy="0" ixz="0"
+                 iyy="2.66739e-7" iyz="0"
+                 izz="9.31478e-7"/>
+      </inertial>
+      <visual>
+        <origin xyz="0 0 0" rpy="0 0 ${M_PI/2}"/>
+        <geometry>
+          <mesh filename="package://phantomx_turret/meshes/F3-Bracket.stl" scale="${M_SCALE} ${M_SCALE} ${M_SCALE}"/>
+        </geometry>
+        <material name="${color}"/>
+      </visual>
+      <collision>
+        <origin xyz="0 0 0" rpy="0 0 0"/>
+        <geometry>
+          <box size="0 0 0"/>
+        </geometry>
+      </collision>
+    </link>
+    <gazebo reference="${name}_link">
+      <material>Gazebo/${color}</material>
+      <selfCollide>true</selfCollide>
+      <gravity>true</gravity>
+    </gazebo>
+  </xacro:macro>
 </robot>

File: urdf/phantomx_turret.urdf.xacro (robot description, xacro)
@@ -31,3 +31,6 @@
     <origin xyz="-2e-6 -9e-6 0.0763" rpy="0 0 0"/>
   </AX12A_compound_fixed>
+  <interbotix_F3_bracket_fixed parent="pan_servo_link" name="pan_F3" color="Gray">
+    <origin xyz="0 0 0.02094" rpy="0 0 0"/>
+  </interbotix_F3_bracket_revolute>
 </robot>

Commit message: Readding tilt servo

File: urdf/pan_tilt_hardware.xacro (robot description, xacro)
@@ -152,41 +152,4 @@
     </gazebo>
   </xacro:macro>
-  <xacro:macro name="interbotix_F3_bracket_revolute" params="parent name color llimit ulimit vlimit elimit *origin">
-    <joint name="${name}_joint" type="revolute">
-      <xacro:insert_block name="origin"/>
-      <axis xyz="0 0 1"/>
-      <limit effort="${elimit}" velocity="${vlimit}" lower="${llimit}" upper="${ulimit}"/>
-      <dynamics friction="0.13"/>
-      <parent link="${parent}"/>
-      <child link="${name}_link"/>
-    </joint>
-    <link name="${name}_link">
-      <inertial>
-        <mass value="0.004398"/>
-        <origin xyz="2.45363e-17 -2.45363e-17 0.00183916"/>
-        <inertia ixx="7.00046e-7" ixy="0" ixz="0"
-                 iyy="2.66739e-7" iyz="0"
-                 izz="9.31478e-7"/>
-      </inertial>
-      <visual>
-        <origin xyz="0 0 0" rpy="0 0 0"/>
-        <geometry>
-          <mesh filename="package://phantomx_turret/meshes/F3-Bracket.stl" scale="${M_SCALE} ${M_SCALE} ${M_SCALE}"/>
-        </geometry>
-        <material name="${color}"/>
-      </visual>
-      <collision>
-        <origin xyz="0 0 0" rpy="0 0 0"/>
-        <geometry>
-          <box size="0 0 0"/>
-        </geometry>
-      </collision>
-    </link>
-    <gazebo reference="${name}_link">
-      <material>Gazebo/${color}</material>
-      <selfCollide>true</selfCollide>
-      <gravity>true</gravity>
-    </gazebo>
-  </xacro:macro>
   <xacro:macro name="interbotix_F3_bracket_fixed" params="parent name color *origin">
     <joint name="${name}_joint" type="fixed">

File: urdf/phantomx_turret.urdf.xacro (robot description, xacro)
@@ -34,3 +34,8 @@
     <origin xyz="0 0 0.02094" rpy="0 0 0"/>
   </interbotix_F3_bracket_fixed>
+  <AX12A_compound_fixed parent="base_mount_link" name="pan_servo"
+                        elimit="${ax12_elimit}" vlimit="${ax12_vlimit}"
+                        llimit="${ax12_llimit}" ulimit="${ax12_ulimit}">
+    <origin xyz="0 0 0.0415" rpy="${M_PI/2} 0 0"/>
+  </AX12A_compound_fixed>
 </robot>

Commit message: Adding F2 bracket

File: urdf/pan_tilt_hardware.xacro (robot description, xacro)
@@ -186,3 +186,37 @@
     </gazebo>
   </xacro:macro>
+  <xacro:macro name="interbotix_F2_bracket_fixed" params="parent name color *origin">
+    <joint name="${name}_joint" type="fixed">
+      <xacro:insert_block name="origin"/>
+      <parent link="${parent}"/>
+      <child link="${name}_link"/>
+    </joint>
+    <link name="${name}_link">
+      <inertial>
+        <mass value="0.011446"/>
+        <origin xyz="-0.00500002 0.0225873 0.00932534"/>
+        <inertia ixx="4.9483e-06" ixy="0" ixz="8.3000e-11"
+                 iyy="2.2081e-06" iyz="0"
+                 izz="4.4637e-06"/>
+      </inertial>
+      <visual>
+        <origin xyz="0 0 0" rpy="0 0 0"/>
+        <geometry>
+          <mesh filename="package://phantomx_turret/meshes/F3-Bracket.stl" scale="${M_SCALE} ${M_SCALE} ${M_SCALE}"/>
+        </geometry>
+        <material name="${color}"/>
+      </visual>
+      <collision>
+        <origin xyz="0 0 0" rpy="0 0 0"/>
+        <geometry>
+          <box size="0 0 0"/>
+        </geometry>
+      </collision>
+    </link>
+    <gazebo reference="${name}_link">
+      <material>Gazebo/${color}</material>
+      <selfCollide>true</selfCollide>
+      <gravity>true</gravity>
+    </gazebo>
+  </xacro:macro>
 </robot>

File: urdf/phantomx_turret.urdf.xacro (robot description, xacro)
@@ -39,3 +39,6 @@
     <origin xyz="0 0 0.0415" rpy="${M_PI/2} 0 0"/>
   </AX12A_compound_fixed>
+  <interbotix_F2_bracket_fixed parent="pan_servo_link" name="pan_F3" color="Gray">
+    <origin xyz="0.005 0.0265 0.024527" rpy="0 0 0"/>
+  </interbotix_F2_bracket_fixed>
 </robot>

Commit message: Adding F2 bracket

File: urdf/pan_tilt_hardware.xacro (robot description, xacro)
@@ -203,5 +203,5 @@
         <origin xyz="0 0 0" rpy="0 0 0"/>
         <geometry>
-          <mesh filename="package://phantomx_turret/meshes/F3-Bracket.stl" scale="${M_SCALE} ${M_SCALE} ${M_SCALE}"/>
+          <mesh filename="package://phantomx_turret/meshes/F2-Bracket.stl" scale="${M_SCALE} ${M_SCALE} ${M_SCALE}"/>
         </geometry>
         <material name="${color}"/>

File: urdf/phantomx_turret.urdf.xacro (robot description, xacro)
@@ -39,5 +39,5 @@
     <origin xyz="0 0 0.0415" rpy="${M_PI/2} 0 ${M_PI/2}"/>
   </AX12A_compound_fixed>
-  <interbotix_F2_bracket_fixed parent="pan_servo_link" name="pan_F3" color="Gray">
+  <interbotix_F2_bracket_fixed parent="tilt_servo_link" name="pan_F2" color="Gray">
     <origin xyz="0.005 0.0265 0.024527" rpy="0 0 0"/>
   </interbotix_F2_bracket_fixed>
