Commit message: Work on F2 Bracket

File: urdf/pan_tilt_hardware.xacro (robot description, xacro)
@@ -201,5 +201,5 @@
       </inertial>
       <visual>
-        <origin xyz="0 0 0" rpy="0 0 0"/>
+        <origin xyz="0 0 0" rpy="${M_PI/2} ${M_PI} 0"/>
         <geometry>
           <mesh filename="package://phantomx_turret/meshes/F2-Bracket.stl" scale="${M_SCALE} ${M_SCALE} ${M_SCALE}"/>

File: urdf/phantomx_turret.urdf.xacro (robot description, xacro)
@@ -40,5 +40,5 @@
   </AX12A_compound_fixed>
   <interbotix_F2_bracket_fixed parent="tilt_servo_link" name="pan_F2" color="Gray">
-    <origin xyz="0.005 0.0265 0.024527" rpy="0 0 0"/>
+    <origin xyz="-0.005 0.0265 0.024527" rpy="0 0 0"/>
   </interbotix_F2_bracket_fixed>
 </robot>

Commit message: Recentering F2

File: urdf/pan_tilt_hardware.xacro (robot description, xacro)
@@ -195,5 +195,5 @@
       <inertial>
         <mass value="0.011446"/>
-        <origin xyz="-0.00500002 0.0225873 0.00932534"/>
+        <origin xyz="1.73681e-8 3.78795e-9 -3.90228e-9"/>
         <inertia ixx="4.9483e-06" ixy="0" ixz="8.3000e-11"
                  iyy="2.2081e-06" iyz="0"

File: urdf/phantomx_turret.urdf.xacro (robot description, xacro)
@@ -40,5 +40,5 @@
   </AX12A_compound_fixed>
   <interbotix_F2_bracket_fixed parent="tilt_servo_link" name="pan_F2" color="Gray">
-    <origin xyz="-0.005 0.0265 0.024527" rpy="0 0 0"/>
+    <origin xyz="-3.601e-7 0.017175 -0.002002" rpy="0 0 0"/>
   </interbotix_F2_bracket_fixed>
 </robot>

Commit message: Added camera mount

File: urdf/pan_tilt_hardware.xacro (robot description, xacro)
@@ -220,3 +220,37 @@
     </gazebo>
   </xacro:macro>
+  <xacro:macro name="camera_mount_fixed" params="parent name color *origin">
+    <joint name="${name}_joint" type="fixed">
+      <xacro:insert_block name="origin"/>
+      <parent link="${parent}"/>
+      <child link="${name}_link"/>
+    </joint>
+    <link name="${name}_link">
+      <inertial>
+        <mass value="0.006453"/>
+        <origin xyz="3.09425e-6 0.00873896 -0.00980897"/>
+        <inertia ixx="1.3618e-06" ixy="1.4400e-10" ixz="8.2000e-11"
+                 iyy="1.4384e-06" iyz="3.8945e-07"
+                 izz="1.5063e-06"/>
+      </inertial>
+      <visual>
+        <origin xyz="0 0 0" rpy="0 0 0"/>
+        <geometry>
+          <mesh filename="package://phantomx_turret/meshes/Head.stl" scale="${M_SCALE} ${M_SCALE} ${M_SCALE}"/>
+        </geometry>
+        <material name="${color}"/>
+      </visual>
+      <collision>
+        <origin xyz="0 0 0" rpy="0 0 0"/>
+        <geometry>
+          <box size="0 0 0"/>
+        </geometry>
+      </collision>
+    </link>
+    <gazebo reference="${name}_link">
+      <material>Gazebo/${color}</material>
+      <selfCollide>true</selfCollide>
+      <gravity>true</gravity>
+    </gazebo>
+  </xacro:macro>
 </robot>

File: urdf/phantomx_turret.urdf.xacro (robot description, xacro)
@@ -42,3 +42,6 @@
     <origin xyz="-3.601e-7 0.017175 -0.002002" rpy="0 0 0"/>
   </interbotix_F2_bracket_fixed>
+  <camera_mount_fixed parent="pan_F2_link" name="camera_mount" color="Gray">
+    <origin xyz="-3.788e-9 0.009325 4e-8" rpy="0 0 0"/>
+  </camera_mount_fixed>
 </robot>

Commit message: Fixed camera mount orientation

File: urdf/pan_tilt_hardware.xacro (robot description, xacro)
@@ -235,5 +235,5 @@
       </inertial>
       <visual>
-        <origin xyz="0 0 0" rpy="0 0 0"/>
+        <origin xyz="0 0 0" rpy="0 ${-M_PI/2} 0"/>
         <geometry>
           <mesh filename="package://phantomx_turret/meshes/Head.stl" scale="${M_SCALE} ${M_SCALE} ${M_SCALE}"/>

Commit message: Adding Camera

File: urdf/pan_tilt_hardware.xacro (robot description, xacro)
@@ -254,3 +254,37 @@
     </gazebo>
   </xacro:macro>
+  <xacro:macro name="rpi_camera_fixed" params="parent name color *origin">
+    <joint name="${name}_joint" type="fixed">
+      <xacro:insert_block name="origin"/>
+      <parent link="${parent}"/>
+      <child link="${name}_link"/>
+    </joint>
+    <link name="${name}_link">
+      <inertial>
+        <mass value="0.003"/>
+        <origin xyz="-0.00911549 -0.012447 0.000734977"/>
+        <inertia ixx="3.5256e-07" ixy="1.1050e-09" ixz="3.5024e-08"
+                 iyy="4.1795e-07" iyz="2.6700e-10"
+                 izz="7.0244e-07"/>
+      </inertial>
+      <visual>
+        <origin xyz="0 0 0" rpy="0 0 0"/>
+        <geometry>
+          <mesh filename="package://phantomx_turret/meshes/Camera.stl" scale="${M_SCALE} ${M_SCALE} ${M_SCALE}"/>
+        </geometry>
+        <material name="${color}"/>
+      </visual>
+      <collision>
+        <origin xyz="0 0 0" rpy="0 0 0"/>
+        <geometry>
+          <box size="0 0 0"/>
+        </geometry>
+      </collision>
+    </link>
+    <gazebo reference="${name}_link">
+      <material>Gazebo/${color}</material>
+      <selfCollide>true</selfCollide>
+      <gravity>true</gravity>
+    </gazebo>
+  </xacro:macro>
 </robot>

File: urdf/phantomx_turret.urdf.xacro (robot description, xacro)
@@ -42,6 +42,9 @@
     <origin xyz="-0.002002 0.017175 -3.601e-7" rpy="0 0 0"/>
   </interbotix_F2_bracket_fixed>
-  <camera_mount_fixed parent="pan_F2_link" name="camera_mount" color="Gray">
+  <camera_mount_fixed parent="pan_F2_link" name="camera_mount" color="White">
     <origin xyz="-3.788e-9 0.009325 4e-8" rpy="0 0 0"/>
   </camera_mount_fixed>
+  <rpi_camera_fixed parent="camera_mount_link" name="camera" color="Green">
+    <origin xyz="-0.0125 0.008 -15.35 mm" rpy="0 0 0"/>
+  </rpi_camera_fixed>
 </robot>

Commit message: Added camera

File: urdf/pan_tilt_hardware.xacro (robot description, xacro)
@@ -269,5 +269,5 @@
       </inertial>
       <visual>
-        <origin xyz="0 0 0" rpy="0 0 0"/>
+        <origin xyz="0 0 0" rpy="${-M_PI/2} 0 ${-M_PI/2}"/>
         <geometry>
           <mesh filename="package://phantomx_turret/meshes/Camera.stl" scale="${M_SCALE} ${M_SCALE} ${M_SCALE}"/>

File: urdf/phantomx_turret.urdf.xacro (robot description, xacro)
@@ -46,5 +46,5 @@
   </camera_mount_fixed>
   <rpi_camera_fixed parent="camera_mount_link" name="camera" color="Green">
-    <origin xyz="-0.0125 0.008 -15.35 mm" rpy="0 0 0"/>
+    <origin xyz="0.01535 0.008 -0.0125" rpy="0 0 0"/>
   </rpi_camera_fixed>
 </robot>

Commit message: Adding camera sensor

File: urdf/pan_tilt_hardware.xacro (robot description, xacro)
@@ -287,4 +287,73 @@
       <gravity>true</gravity>
     </gazebo>
+    <joint name="${name}_lens_joint" type="fixed">
+      <origin xyz="-0.009462 -0.0125 0.00615" rpy="0 0 0"/>
+      <parent link="${name}_link"/>
+      <child link="${name}_lens_link"/>
+    </joint>
+    <link name="${name}_link">
+      <inertial>
+        <mass value="0.0001"/>
+        <origin xyz="0 0 0"/>
+        <inertia ixx="1e-09" ixy="0" ixz="0"
+                 iyy="1e-09" iyz="0"
+                 izz="1e-09"/>
+      </inertial>
+      <visual>
+        <origin xyz="0 0 0" rpy="0 0 0"/>
+        <geometry>
+          <cylinder radius="0.0005" length="0.0005"/>
+        </geometry>
+        <material name="Black"/>
+      </visual>
+      <collision>
+        <origin xyz="0 0 0" rpy="0 0 0"/>
+        <geometry>
+          <box size="0 0 0"/>
+        </geometry>
+      </collision>
+    </link>
+    <gazebo reference="${name}_lens_link">
+      <material>Gazebo/Black</material>
+      <selfCollide>true</selfCollide>
+      <gravity>true</gravity>
+      <sensor type="camera" name="${name}_camera">
+        <update_rate>15.0</update_rate>
+        <camera name="camera">
+          <horizontal_fov>${62.2 * M_PI/180.0}</horizontal_fov>
+          <image>
+            <width>3240</width>
+            <height>2464</height>
+            <format>R8G8B8</format>
+          </image>
+          <clip>
+            <near>0.02</near>
+            <far>300</far>
+          </clip>
+          <noise>
+            <type>gaussian</type>
+            <!-- Noise is sampled independently per pixel on each frame.
+                That pixel's noise value is added to each of its color
+                channels, which at that point lie in the range [0,1]. -->
+            <mean>0.0</mean>
+            <stddev>0.007</stddev>
+          </noise>
+        </camera>
+        <plugin name="camera_controller" filename="libgazebo_ros_camera.so">
+          <alwaysOn>true</alwaysOn>
+          <updateRate>0.0</updateRate>
+          <cameraName>phantomx_turret/camera</cameraName>
+          <imageTopicName>image_raw</imageTopicName>
+          <cameraInfoTopicName>camera_info</cameraInfoTopicName>
+          <frameName>${name}_lens_link</frameName>
+          <hackBaseline>0.07</hackBaseline>
+          <distortionK1>0.0</distortionK1>
+          <distortionK2>0.0</distortionK2>
+          <distortionK3>0.0</distortionK3>
+          <distortionT1>0.0</distortionT1>
+          <distortionT2>0.0</distortionT2>
+        </plugin>
+      </sensor>
+    </gazebo>
   </xacro:macro>
 </robot>

Commit message: Fixed position of camera lens

File: urdf/pan_tilt_hardware.xacro (robot description, xacro)
@@ -288,9 +288,9 @@
     </gazebo>
     <joint name="${name}_lens_joint" type="fixed">
-      <origin xyz="-0.009462 -0.0125 0.00615" rpy="0 0 0"/>
+      <origin xyz="0.00615 0.009462 0.0125" rpy="0 0 0"/>
       <parent link="${name}_link"/>
       <child link="${name}_lens_link"/>
     </joint>
-    <link name="${name}_link">
+    <link name="${name}_lens_link">
       <inertial>
         <mass value="0.0001"/>
@@ -301,5 +301,5 @@
       </inertial>
       <visual>
-        <origin xyz="0 0 0" rpy="0 0 0"/>
+        <origin xyz="0 0 0" rpy="0 ${M_PI/2} 0"/>
         <geometry>
           <cylinder radius="0.0005" length="0.0005"/>

Commit message: Getting model to work in gazebo

File: urdf/pan_tilt_hardware.xacro (robot description, xacro)
@@ -13,6 +13,6 @@
         <mass value="0.21328"/>
         <origin xyz="0.00199427 0.0257168 0.00107065"/>
-        <inertia ixx="0.0003798" ixy="-6.70148E-7" ixz="-5.778745E-6"
-                 iyy="0.0006116" iyz="-8.17711E-7"
+        <inertia ixx="0.0003798" ixy="0" ixz="0"
+                 iyy="0.0006116" iyz="0"
                  izz="0.000379"/>
       </inertial>
@@ -25,5 +25,5 @@
       </visual>
       <collision>
-        <origin xyz="-2e-6 0.05785 -9e-6" rpy="0 0 0"/>
+        <origin xyz="-2e-6 -9e-6 0.05785" rpy="${M_PI/2} 0 0"/>
         <geometry>
           <box size="0.1045 0.0049 0.1045"/>
@@ -31,5 +31,5 @@
       </collision>
       <collision>
-        <origin xyz="-2e-6 0.0329 -9.5e-6" rpy="0 0 0"/>
+        <origin xyz="-2e-6 -9.5e-6 0.0329" rpy="${M_PI/2} 0 0"/>
         <geometry>
           <box size="0.086 0.045 0.086929"/>
@@ -37,5 +37,5 @@
       </collision>
       <collision>
-        <origin xyz="-2e-6 0.005139 -9e-6" rpy="0 0 0"/>
+        <origin xyz="-2e-6 -9e-6 0.005139" rpy="${M_PI/2} 0 0"/>
         <geometry>
           <box size="0.178 0.010522 0.178"/>
@@ -45,5 +45,5 @@
     <gazebo reference="${name}_link">
       <material>Gazebo/${color}</material>
-      <selfCollide>true</selfCollide>
+      <selfCollide>false</selfCollide>
       <gravity>true</gravity>
     </gazebo>
@@ -79,5 +79,5 @@
     <gazebo reference="${name}_link">
       <material>Gazebo/Black</material>
-      <selfCollide>true</selfCollide>
+      <selfCollide>false</selfCollide>
       <gravity>true</gravity>
     </gazebo>
@@ -107,5 +107,5 @@
         <origin xyz="0 0 0" rpy="0 0 0"/>
         <geometry>
-          <box size="0 0 0"/>
+          <box size="0.001 0.001 0.001"/>
         </geometry>
       </collision>
@@ -113,5 +113,5 @@
     <gazebo reference="${name}_body_link">
       <material>Gazebo/Black</material>
-      <selfCollide>true</selfCollide>
+      <selfCollide>false</selfCollide>
       <gravity>true</gravity>
     </gazebo>
@@ -142,5 +142,5 @@
         <origin xyz="0 0 0" rpy="0 0 0"/>
         <geometry>
-          <box size="0 0 0"/>
+          <box size="0.001 0.001 0.001"/>
         </geometry>
       </collision>
@@ -148,5 +148,5 @@
     <gazebo reference="${name}_link">
       <material>Gazebo/Black</material>
-      <selfCollide>true</selfCollide>
+      <selfCollide>false</selfCollide>
       <gravity>true</gravity>
     </gazebo>
@@ -176,11 +176,11 @@
         <origin xyz="0 0 0" rpy="0 0 0"/>
         <geometry>
-          <box size="0 0 0"/>
-        </geometry>
-      </collision>
-    </link>
-    <gazebo reference="${name}_link">
-      <material>Gazebo/${color}</material>
-      <selfCollide>true</selfCollide>
+          <box size="0.001 0.001 0.001"/>
+        </geometry>
+      </collision>
+    </link>
+    <gazebo reference="${name}_link">
+      <material>Gazebo/${color}</material>
+      <selfCollide>false</selfCollide>
       <gravity>true</gravity>
     </gazebo>
@@ -210,11 +210,11 @@
         <origin xyz="0 0 0" rpy="0 0 0"/>
         <geometry>
-          <box size="0 0 0"/>
-        </geometry>
-      </collision>
-    </link>
-    <gazebo reference="${name}_link">
-      <material>Gazebo/${color}</material>
-      <selfCollide>true</selfCollide>
+          <box size="0.001 0.001 0.001"/>
+        </geometry>
+      </collision>
+    </link>
+    <gazebo reference="${name}_link">
+      <material>Gazebo/${color}</material>
+      <selfCollide>false</selfCollide>
       <gravity>true</gravity>
     </gazebo>
@@ -244,11 +244,11 @@
         <origin xyz="0 0 0" rpy="0 0 0"/>
         <geometry>
-          <box size="0 0 0"/>
-        </geometry>
-      </collision>
-    </link>
-    <gazebo reference="${name}_link">
-      <material>Gazebo/${color}</material>
-      <selfCollide>true</selfCollide>
+          <box size="0.001 0.001 0.001"/>
+        </geometry>
+      </collision>
+    </link>
+    <gazebo reference="${name}_link">
+      <material>Gazebo/${color}</material>
+      <selfCollide>false</selfCollide>
       <gravity>true</gravity>
     </gazebo>
@@ -278,11 +278,11 @@
         <origin xyz="0 0 0" rpy="0 0 0"/>
         <geometry>
-          <box size="0 0 0"/>
-        </geometry>
-      </collision>
-    </link>
-    <gazebo reference="${name}_link">
-      <material>Gazebo/${color}</material>
-      <selfCollide>true</selfCollide>
+          <box size="0.001 0.001 0.001"/>
+        </geometry>
+      </collision>
+    </link>
+    <gazebo reference="${name}_link">
+      <material>Gazebo/${color}</material>
+      <selfCollide>false</selfCollide>
       <gravity>true</gravity>
     </gazebo>
@@ -308,7 +308,7 @@
       </visual>
       <collision>
-        <origin xyz="0 0 0" rpy="0 0 0"/>
-        <geometry>
-          <box size="0 0 0"/>
+        <origin xyz="0 0 0" rpy="0 ${M_PI/2} 0"/>
+        <geometry>
+          <cylinder radius="0.0005" length="0.0005"/>
         </geometry>
       </collision>
@@ -316,5 +316,5 @@
     <gazebo reference="${name}_lens_link">
       <material>Gazebo/Black</material>
-      <selfCollide>true</selfCollide>
+      <selfCollide>false</selfCollide>
       <gravity>true</gravity>
       <sensor type="camera" name="${name}_camera">

Commit message: Fixed urdf files Fixed a bunch of arduino errors Added teleop script

File: urdf/pan_tilt_hardware.xacro (robot description, xacro)
@@ -4,5 +4,5 @@
   <xacro:property name="M_SCALE" value="0.001"/>
   <xacro:macro name="base_mount" params="parent name color *origin">
-    <joint name="${name}_joint" type="fixed">
+   <joint name="${name}_joint" type="fixed">
       <xacro:insert_block name="origin"/>
         <parent link="${parent}"/>

File: urdf/phantomx_turret.urdf.xacro (robot description, xacro)
@@ -21,7 +21,6 @@
     <color rgba="0.22 0.32 0.14 1.0"/>
   </material>
-  <!-- Used for fixing robot to Gazebo 'base_link' -->
-  <link name="world"/>
-  <base_mount parent="world" name="base_mount" color="Gray" >
+  <link name="base_link"/>
+  <base_mount parent="base_link" name="base_mount" color="Gray" >
       <origin xyz="0 0 0" rpy="0 0 0"/>
   </base_mount>
